File: OpenSprinkler Pi/hardware/ospi_v10.brd (EAGLE design)
At the start: 99.9 x 73.7 mm, 45 parts, among them IC1 MC33063/MC34063D, IC3 DS1307, IC5 74HC595N, J0 24VAC IN, J2 EG1206, T1 MAC97, T2 MAC97, T3 MAC97, T4 MAC97, T5 MAC97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

Commit message: fix component values
Parts:
- removed C6: 0.1u, rcl:C0805
- added C3, C4: 0.1u, rcl:C0805
- added L1: 100uH, SparkFunNew:SRU1038
- CT: value 220p -> 68pF
- D1: value S1A -> R3000
- D2: device diode:DO214AC -> diode:DO-214AC
- L1': device SparkFunNew:SRU1038 -> rcl:6000-XXXX-RC
- RLED: value 30K -> 330
- moved L1' 3.89 mm to (35.1, 15.5), turned to 270 degrees
- moved X3 2.27 mm to (54.4, 55.6), turned to 90 degrees
- moved D2 1.93 mm to (33.5, 27.2)
- moved JP1 1.27 mm to (29.0, 67.3)
- moved RCL 0.76 mm to (57.9, 63.8), turned to 0 degrees
- moved ROE 0.76 mm to (39.9, 54.6)
- moved PWR_LED 0.76 mm to (4.06, 43.4), turned to 270 degrees
- moved CT 0.57 mm to (29.7, 24.6)
- moved RDA 0.51 mm to (61.7, 63.8), turned to 180 degrees
- moved J0 0.51 mm to (1.52, 17.8)
- moved JP2 0.51 mm to (81.0, 67.3)
- moved RLED 0.51 mm to (4.06, 40.9), turned to 180 degrees
- moved J2 0.25 mm to (2.29, 28.8)
Connections:
- net GND: now also C3.2, C4.2; no longer C6.2
- net N$46: now also L1.1
- net VCC: now also C3.1
- net VIN: now also C4.1; no longer C6.1
- net VIN_PRE: now also L1.2
Routing:
- net GND: track 369.0 -> 0.00 mm
- net VIN: track 195.3 -> 142.1 mm
- net D7: track 139.9 -> 104.2 mm, vias 1 -> 2
- net VCC: track 118.0 -> 96.1 mm
- net A1: track 122.0 -> 101.9 mm, vias 0 -> 1
- net QH*: track 64.0 -> 57.7 mm, vias 1 -> 2
- net N$2: track 28.1 -> 34.1 mm
- net N$27: track 29.8 -> 35.6 mm, vias 2 -> 0
- net N$14: track 18.7 -> 14.7 mm
- net N$16: track 36.0 -> 32.5 mm
- net SCL: track 33.3 -> 30.7 mm, vias 1 -> 0
- net N$18: track 32.6 -> 35.1 mm, vias 1 -> 0
- net N$47: track 6.22 -> 3.93 mm
- net N$46: track 13.7 -> 15.9 mm
- net N$29: track 38.0 -> 39.8 mm, vias 2 -> 0
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Other:
- board text added: "Rayshobby, 02/2013"
- board text removed: "Rayshobby, 01/2013"
