File: OpenSprinkler Pi/hardware/ospi_v10.sch (EAGLE design)
At the start: 45 parts, among them IC1 MC33063/MC34063D, IC3 DS1307, IC5 74HC595N, J0 24VAC IN, J2 EG1206, T1 MAC97, T2 MAC97, T3 MAC97, T4 MAC97, T5 MAC97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

Commit message: fix component values
Parts:
- added C3: 0.1u, rcl:C-EUC0805
- added L1: 100uH, SparkFunNew:INDUCTORSRU1038
- CT: value 220p -> 68pF
- D1: value S1A -> R3000
- D2: device diode:DIODE-DO214AC -> diode:DIODE-DO-214AC
- L1': device SparkFunNew:INDUCTORSRU1038 -> rcl:L-US6000-XXX-RC
- RLED: value 30K -> 330
- renumbered C6 to C4
Connections:
- net GND: now also C3.2
- net N$46: now also L1.1
- net VCC: now also C3.1
- net VIN_PRE: now also L1.2
Changed lines of the file:
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@@
 <clearance class="0" value="0.2032"/>
 </class>
-<class number="1" name="power" width="0.762" drill="0">
+<class number="1" name="power" width="0.6096" drill="0">
 <clearance class="1" value="0.2032"/>
 </class>
@@
 <part name="P+2" library="supply1" deviceset="VCC" device=""/>
 <part name="C1" library="resistor" deviceset="CPOL-EU" device="E3.5-8" value="100u"/>
-<part name="D2" library="diode" deviceset="DIODE-" device="DO214AC" value="SS14"/>
+<part name="D2" library="diode" deviceset="DIODE-" device="DO-214AC" value="SS14"/>
 <part name="C2" library="resistor" deviceset="CPOL-EU" device="E3.5-8" value="470u"/>
-<part name="D1" library="diode" deviceset="DIODE-" device="DO41-7.6" value="S1A"/>
+<part name="D1" library="diode" deviceset="DIODE-" device="DO41-7.6" value="R3000"/>
 <part name="GND6" library="SparkFun" deviceset="GND" device=""/>
 <part name="J2" library="adafruit" deviceset="EG1206" device=""/>
 <part name="IC1" library="adafruit" deviceset="MC33063/MC34063" device="D"/>
 <part name="RSC" library="rcl" deviceset="R-EU_" device="R0805" value="1.0"/>
-<part name="CT" library="rcl" deviceset="C-EU" device="C0805" value="220p"/>
+<part name="CT" library="rcl" deviceset="C-EU" device="C0805" value="68pF"/>
 <part name="RT" library="rcl" deviceset="R-EU_" device="R0805" value="30K"/>
 <part name="RB" library="rcl" deviceset="R-EU_" device="R0805" value="10K"/>
@@
 <part name="RCL" library="rcl" deviceset="R-EU_" device="R0805" value="10K"/>
 <part name="RDA" library="rcl" deviceset="R-EU_" device="R0805" value="10K"/>
-<part name="C6" library="rcl" deviceset="C-EU" device="C0805" value="0.1u"/>
+<part name="C4" library="rcl" deviceset="C-EU" device="C0805" value="0.1u"/>
 <part name="GND10" library="SparkFun" deviceset="GND" device=""/>
 <part name="RN2" library="resistor-dil" deviceset="4R-N" device="EXB38V"/>
 <part name="RN3" library="resistor-dil" deviceset="4R-N" device="EXB38V"/>
 <part name="X3" library="crystal" deviceset="CRYSTAL" device="TC26H" value="32.657k"/>
-<part name="L1'" library="SparkFunNew" deviceset="INDUCTOR" device="SRU1038" value="220uH"/>
+<part name="L1" library="SparkFunNew" deviceset="INDUCTOR" device="SRU1038" value="100uH"/>
 <part name="RSC1" library="rcl" deviceset="R-EU_" device="R0805" value="1.0"/>
 <part name="EXTOUT1" library="pinhead" deviceset="PINHD-2X4" device="/90"/>
@@
 <part name="D3" library="diode" deviceset="DIODE-" device="DO34-7" value="5.1V"/>
 <part name="PWR_LED" library="adafruit" deviceset="LED" device="CHIPLED_0805"/>
-<part name="RLED" library="rcl" deviceset="R-EU_" device="R0805" value="30K"/>
+<part name="RLED" library="rcl" deviceset="R-EU_" device="R0805" value="330"/>
 <part name="JP1" library="SparkFunNew" deviceset="M08" device="LOCK"/>
 <part name="JP2" library="SparkFun" deviceset="M03" device="LOCK"/>
 <part name="U$2" library="RaspberryPi" deviceset="OSPI" device=""/>
+<part name="L1'" library="rcl" deviceset="L-US" device="6000-XXX-RC" value="220uH"/>
+<part name="C3" library="rcl" deviceset="C-EU" device="C0805" value="0.1u"/>
+<part name="GND1" library="SparkFun" deviceset="GND" device=""/>
 </parts>
 <sheets>
@@
 </instance>
 <instance part="RSC" gate="G$1" x="59.69" y="154.94" smashed="yes" rot="MR270">
-<attribute name="NAME" x="60.96" y="159.7914" size="1.778" layer="95" rot="MR180"/>
+<attribute name="NAME" x="64.77" y="159.7914" size="1.778" layer="95" rot="MR180"/>
+<attribute name="VALUE" x="64.77" y="156.972" size="1.778" layer="96" rot="MR180"/>
 </instance>
 <instance part="CT" gate="G$1" x="24.13" y="129.54" smashed="yes">
@@
 <attribute name="VALUE" x="135.89" y="143.002" size="1.778" layer="96" rot="MR180"/>
 </instance>
-<instance part="C6" gate="G$1" x="137.16" y="158.75" smashed="yes">
+<instance part="C4" gate="G$1" x="137.16" y="158.75" smashed="yes">
 <attribute name="NAME" x="131.064" y="156.591" size="1.778" layer="95"/>
 <attribute name="VALUE" x="131.064" y="154.051" size="1.778" layer="96"/>
@@
 <attribute name="VALUE" x="161.29" y="158.75" size="1.778" layer="96" rot="MR0"/>
 </instance>
-<instance part="L1'" gate="G$1" x="76.2" y="157.48" smashed="yes"/>
-<instance part="RSC1" gate="G$1" x="62.23" y="154.94" smashed="yes" rot="MR270">
-<attribute name="NAME" x="63.5" y="159.7914" size="1.778" layer="95" rot="MR180"/>
-</instance>
+<instance part="L1" gate="G$1" x="76.2" y="157.48" smashed="yes">
+<attribute name="NAME" x="78.74" y="162.56" size="1.778" layer="95"/>
+<attribute name="VALUE" x="78.74" y="160.02" size="1.778" layer="96"/>
+</instance>
+<instance part="RSC1" gate="G$1" x="62.23" y="154.94" smashed="yes" rot="MR270"/>
 <instance part="EXTOUT1" gate="A" x="27.94" y="10.16"/>
-<instance part="RSC2" gate="G$1" x="57.15" y="154.94" smashed="yes" rot="MR270">
-<attribute name="NAME" x="58.42" y="159.7914" size="1.778" layer="95" rot="MR180"/>
-</instance>
+<instance part="RSC2" gate="G$1" x="57.15" y="154.94" smashed="yes" rot="MR270"/>
 <instance part="F1" gate="G$1" x="93.98" y="149.86" rot="R180"/>
 <instance part="D3" gate="G$1" x="99.06" y="135.89" rot="R90"/>
@@
 <instance part="JP2" gate="G$1" x="119.38" y="67.31"/>
 <instance part="U$2" gate="G$1" x="172.72" y="66.04"/>
+<instance part="L1'" gate="G$1" x="73.66" y="157.48" smashed="yes"/>
+<instance part="C3" gate="G$1" x="35.56" y="67.31" smashed="yes">
+<attribute name="NAME" x="29.464" y="65.151" size="1.778" layer="95"/>
+<attribute name="VALUE" x="29.464" y="62.611" size="1.778" layer="96"/>
+</instance>
+<instance part="GND1" gate="1" x="35.56" y="59.69"/>
 </instances>
 <busses>
@@
 </busses>
 <nets>
-<net name="GND" class="0">
+<net name="GND" class="1">
 <segment>
 <wire x1="71.12" y1="86.36" x2="78.74" y2="86.36" width="0.1524" layer="91"/>
@@
 </segment>
 <segment>
-<pinref part="C6" gate="G$1" pin="2"/>
+<pinref part="C4" gate="G$1" pin="2"/>
 <pinref part="GND10" gate="1" pin="GND"/>
 </segment>
@@
 <wire x1="127" y1="64.77" x2="139.7" y2="64.77" width="0.1524" layer="91"/>
 <label x="133.35" y="64.77" size="1.778" layer="95"/>
+</segment>
+<segment>
+<pinref part="C3" gate="G$1" pin="2"/>
+<pinref part="GND1" gate="1" pin="GND"/>
 </segment>
 </net>
@@
 <pinref part="IC3" gate="G$1" pin="VCC"/>
 <pinref part="RCL" gate="G$1" pin="1"/>
-<pinref part="C6" gate="G$1" pin="1"/>
+<pinref part="C4" gate="G$1" pin="1"/>
 </segment>
 <segment>
@@
 <wire x1="41.91" y1="69.85" x2="41.91" y2="53.34" width="0.1524" layer="91"/>
 <wire x1="15.24" y1="45.72" x2="15.24" y2="69.85" width="0.1524" layer="91"/>
-<wire x1="15.24" y1="69.85" x2="41.91" y2="69.85" width="0.1524" layer="91"/>
+<wire x1="15.24" y1="69.85" x2="35.56" y2="69.85" width="0.1524" layer="91"/>
+<wire x1="35.56" y1="69.85" x2="41.91" y2="69.85" width="0.1524" layer="91"/>
 <wire x1="15.24" y1="45.72" x2="16.51" y2="45.72" width="0.1524" layer="91"/>
 <junction x="41.91" y="69.85"/>
@@
 <pinref part="P+2" gate="VCC" pin="VCC"/>
 <pinref part="ROE" gate="G$1" pin="2"/>
+<pinref part="C3" gate="G$1" pin="1"/>
+<junction x="35.56" y="69.85"/>
 </segment>
 <segment>
@@
 <wire x1="21.59" y1="154.94" x2="25.4" y2="154.94" width="0.1524" layer="91"/>
 <wire x1="21.59" y1="154.94" x2="21.59" y2="167.64" width="0.1524" layer="91"/>
-<wire x1="21.59" y1="167.64" x2="76.2" y2="167.64" width="0.1524" layer="91"/>
+<wire x1="21.59" y1="167.64" x2="73.66" y2="167.64" width="0.1524" layer="91"/>
 <junction x="21.59" y="154.94"/>
 <pinref part="D2" gate="G$1" pin="C"/>
 <pinref part="IC1" gate="G$1" pin="SWE"/>
+<pinref part="L1" gate="G$1" pin="1"/>
+<wire x1="73.66" y1="167.64" x2="76.2" y2="167.64" width="0.1524" layer="91"/>
+<wire x1="76.2" y1="167.64" x2="76.2" y2="165.1" width="0.1524" layer="91"/>
 <pinref part="L1'" gate="G$1" pin="1"/>
-<wire x1="76.2" y1="167.64" x2="76.2" y2="165.1" width="0.1524" layer="91"/>
+<wire x1="73.66" y1="165.1" x2="73.66" y2="167.64" width="0.1524" layer="91"/>
+<junction x="73.66" y="167.64"/>
 </segment>
 </net>
@@
 <wire x1="76.2" y1="149.86" x2="76.2" y2="132.08" width="0.1524" layer="91"/>
 <wire x1="86.36" y1="149.86" x2="76.2" y2="149.86" width="0.1524" layer="91"/>
-<wire x1="64.77" y1="149.86" x2="76.2" y2="149.86" width="0.1524" layer="91"/>
+<wire x1="64.77" y1="149.86" x2="73.66" y2="149.86" width="0.1524" layer="91"/>
 <junction x="76.2" y="149.86"/>
 <label x="77.47" y="147.32" size="1.778" layer="95"/>
 <pinref part="C2" gate="G$1" pin="+"/>
 <pinref part="RT" gate="G$1" pin="1"/>
+<pinref part="L1" gate="G$1" pin="2"/>
+<pinref part="F1" gate="G$1" pin="2"/>
 <pinref part="L1'" gate="G$1" pin="2"/>
-<pinref part="F1" gate="G$1" pin="2"/>
-</segment>
-</net>
+<wire x1="73.66" y1="149.86" x2="76.2" y2="149.86" width="0.1524" layer="91"/>
+<junction x="73.66" y="149.86"/>
+</segment>
+</net>
