File: OpenSprinkler Controller/hardware/v2.3/DC/os23dc.sch (EAGLE design)
At the start: 121 parts, among them J1 POWER, Q1 BSS123, Q2 BSS123, Q3 BSS123, Q4 BSS123, Q5 BSS123, Q6 BSS123, Q7 BSS123, Q8 BSS123, X0 32.768kHz

Commit message: correct some component values
Parts:
- CT: value 470 -> 330pF
- L1': value 1000uH -> 220uH
- Q1: value BSS123 -> AO3400
- QB1: value (none) -> 2N3904
- QP1: value BSS84 -> AP3401
- R0: value 3.3ohm -> 1ohm
- RB: value 1.5K -> 1.6K
- RSC: value 3.3 -> 1
- RT: value 25K -> 27K
- RZ: value 180 -> 100
Other:
- note removed: "330x4 Isolated ResNet"
